Commit message: making updates before checkin to master

File: my_robot/urdf/my_robot.xacro (robot description, xacro)
@@ -31,28 +31,4 @@
       </geometry>
     </visual>
-    <collision name='back_caster_collision'>
-      <origin xyz="-0.15 0 -0.05" rpy=" 0 0 0"/>
-      <geometry>
-        <sphere radius="0.0499"/>
-      </geometry>
-    </collision>
-    <visual name='back_caster_visual'>
-      <origin xyz="-0.15 0 -0.05" rpy=" 0 0 0"/>
-      <geometry>
-        <sphere radius="0.05"/>
-      </geometry>
-    </visual>
-    <collision name='front_caster_collision'>
-      <origin xyz="0.15 0 -0.05" rpy=" 0 0 0"/>
-      <geometry>
-        <sphere radius="0.0499"/>
-      </geometry>
-    </collision>
-    <visual name='front_caster_visual'>
-      <origin xyz="0.15 0 -0.05" rpy=" 0 0 0"/>
-      <geometry>
-        <sphere radius="0.05"/>
-      </geometry>
-    </visual>
   </link>
   <link name='left_wheel'>
@@ -96,4 +72,50 @@
     </collision>
     <visual name='right_wheel_visual'>
+      <origin xyz="0 0 0" rpy="0 1.5707 1.5707"/>
+      <geometry>
+        <cylinder length="0.05" radius = ".1"/>
+      </geometry>
+    </visual>
+  </link>
+  <link name='left_rear_wheel'>
+    <inertial>
+      <mass value="5.0"/>
+      <origin xyz="0 0 0" rpy=" 0 1.5707 1.5707"/>
+      <inertia
+          ixx="0.1" ixy="0" ixz="0"
+          iyy="0.1" iyz="0"
+          izz="0.1"
+      />
+    </inertial>
+    <collision name='left_rear_wheel_collision'>
+      <origin xyz="0 0 0" rpy="0 1.5707 1.5707"/>
+      <geometry>
+        <cylinder length="0.05" radius = ".1"/>
+      </geometry>
+    </collision>
+    <visual name='left_rear_wheel_visual'>
+      <origin xyz="0 0 0" rpy="0 1.5707 1.5707"/>
+      <geometry>
+        <cylinder length="0.05" radius = ".1"/>
+      </geometry>
+    </visual>
+  </link>
+  <link name='right_rear_wheel'>
+    <inertial>
+      <mass value="5.0"/>
+      <origin xyz="0 0 0" rpy=" 0 1.5707 1.5707"/>
+      <inertia
+          ixx="0.1" ixy="0" ixz="0"
+          iyy="0.1" iyz="0"
+          izz="0.1"
+      />
+    </inertial>
+    <collision name='right_rear_wheel_collision'>
+      <origin xyz="0 0 0" rpy="0 1.5707 1.5707"/>
+      <geometry>
+        <cylinder length="0.05" radius = ".1"/>
+      </geometry>
+    </collision>
+    <visual name='right_rear_wheel_visual'>
       <origin xyz="0 0 0" rpy="0 1.5707 1.5707"/>
       <geometry>
@@ -164,4 +186,20 @@
     <dynamics damping="1.0" friction="1.0"/>
   </joint>
+  <joint type="continuous" name="left_rear_wheel_hinge">
+    <origin xyz="-.2 0.15 0" rpy="0 0 0"/>
+    <child link="left_rear_wheel"/>
+    <parent link="chassis"/>
+    <axis xyz="0 1 0" rpy="0 0 0"/>
+    <limit effort="10000" velocity="1000"/>
+    <dynamics damping="1.0" friction="0.1"/>
+  </joint>
+  <joint type="continuous" name="right_rear_wheel_hinge">
+    <origin xyz="-.2 -0.15 0" rpy="0 0 0"/>
+    <child link="right_rear_wheel"/>
+    <parent link="chassis"/>
+    <axis xyz="0 1 0" rpy="0 0 0"/>
+    <limit effort="10000" velocity="1000"/>
+    <dynamics damping="1.0" friction="0.1"/>
+  </joint>
   <joint type="fixed" name="camera_joint">
     <origin xyz="0.2 0 0" rpy="0 0 0"/>
@@ -180,3 +218,23 @@
     <dynamics damping="1.0" friction="1.0"/>
   </joint>
+  <!--transmission name="right_side_wheel_trans">
+      <type>pr2_mechanism_model/SimpleTransmission</type>
+      <actuator name="right_motor_link">
+        <mechanicalReduction>1.0</mechanicalReduction>
+        <motorTorqueConstant>1</motorTorqueConstant>
+      </actuator>
+      <joint name="right_wheel_hinge">
+        <hardwareInterface>EffortJointInterface</hardwareInterface>
+      </joint>
+  </transmission-->
+  <!--transmission name="left_side_wheel_trans">
+      <type>pr2_mechanism_model/SimpleTransmission</type>
+      <actuator name="left_motor_link">
+        <mechanicalReduction>1.0</mechanicalReduction>
+        <motorTorqueConstant>1</motorTorqueConstant>
+      </actuator>
+      <joint name="left_wheel_hinge">
+        <hardwareInterface>EffortJointInterface</hardwareInterface>
+      </joint>
+  </transmission-->
 </robot>

Commit message: added color to the base

File: my_robot/urdf/my_robot.xacro (robot description, xacro)
@@ -2,4 +2,5 @@
 <robot name="my_robot" xmlns:xacro="http://www.ros.org/wiki/xacro">
   <xacro:include filename="$(find my_robot)/urdf/my_robot.gazebo" />
+  <xacro:include filename="$(find my_robot)/urdf/materials.xacro" />
   <link name="robot_footprint"></link>
   <joint name="robot_footprint_joint" type="fixed">
@@ -32,4 +33,7 @@
     </visual>
   </link>
+  <gazebo reference="chassis">
+    <material>Gazebo/Red</material>
+  </gazebo>
   <link name='left_wheel'>
     <inertial>
@@ -53,4 +57,5 @@
         <cylinder length="0.05" radius = ".1"/>
       </geometry>
+      <material name="orange"/>
     </visual>
   </link>

Commit message: changed some more colors

File: my_robot/urdf/my_robot.xacro (robot description, xacro)
@@ -60,4 +60,7 @@
     </visual>
   </link>
+  <gazebo reference="left_wheel">
+    <material>Gazebo/Grey</material>
+  </gazebo>
   <link name='right_wheel'>
     <inertial>
@@ -83,4 +86,7 @@
     </visual>
   </link>
+  <gazebo reference="right_wheel">
+    <material>Gazebo/Grey</material>
+  </gazebo>
   <link name='left_rear_wheel'>
     <inertial>
@@ -106,4 +112,7 @@
     </visual>
   </link>
+  <gazebo reference="left_rear_wheel">
+    <material>Gazebo/Black</material>
+  </gazebo>
   <link name='right_rear_wheel'>
     <inertial>
@@ -129,4 +138,7 @@
     </visual>
   </link>
+  <gazebo reference="right_rear_wheel">
+    <material>Gazebo/Black</material>
+  </gazebo>
   <link name='camera'>
     <inertial>

Commit message: checking ability to change hokuyo mesh color

File: my_robot/urdf/my_robot.xacro (robot description, xacro)
@@ -187,4 +187,7 @@
     </visual>
   </link>
+  <gazebo reference="hokuyo">
+    <material>Gazebo/Green</material>
+  </gazebo>
   <joint type="continuous" name="left_wheel_hinge">
     <origin xyz="0 0.15 0" rpy="0 0 0"/>
